Commit message: feat: 机械臂视觉抓取，采用 GRCNN 方案

File: src/urdf/urdf/DM_urdf.urdf (robot description, URDF)
Before this commit: robot DM_urdf, 7 links, 6 joints
Links:
- added link tool0_tcp; visual sphere radius=0.005
Joints:
- added joint joint_tcp: type fixed, parent link_6, child tool0_tcp, origin xyz=0 0 0.16 rpy=0 0 0
